File: hss.kicad_sch (KiCad schematic)
At the start: 4 parts, among them U17 BTS6143D

Commit message: added footprints to almost all components
Parts:
- D11: footprint (none) -> Package_TO_SOT_SMD:SOT-23_Handsoldering; Mouser# (none) -> 771-PLVA650A-QR
- R26, R30: footprint (none) -> Resistor_SMD:R_0805_2012Metric_Pad1.20x1.40mm_HandSolder
