File: hss.kicad_sch (KiCad schematic)
At the start: 8 parts, among them J20 Conn_01x04, U17 BTS6143D

Commit message: bajs
Parts:
- renumbered D32 to D1, D11 to D26, J20 to J3, R112 to R18, R64 to R3, R30 to R70, R26 to R72, U17 to U27
