File: launchpad-controller-v2.kicad_sch (KiCad schematic)
At the start: 49 parts, among them J5 Screw_Terminal_01x02, U13 STM32H723ZGTx, U21 74LS06, U22 74LS06, Y1 50MHz, Y2 32.768 kHz

Commit message: Launchpad controller revision 06/03/2024
Parts:
- added BT1: Battery_Cell, Battery:Battery_Panasonic_CR2032-VS1N_Vertical_CircularHoles, symbol Device:Battery_Cell
- added C102: 22u, symbol Device:C
- added C104, C105: 100n, symbol Device:C
- added D29, D30, D31: 5V, symbol Device:D_Zener
- added J16, J18, J19, J20, J21: Conn_01x02_Socket, symbol Connector:Conn_01x02_Socket
- added J23: Conn_ST_STDC14, Connector_PinHeader_1.27mm:PinHeader_2x07_P1.27mm_Vertical_SMD, symbol Connector:Conn_ST_STDC14
- added J31, J32, J33: Conn_01x12_Pin, Connector_PinHeader_2.54mm:PinHeader_1x12_P2.54mm_Vertical, symbol Connector:Conn_01x12_Pin
- added J42: Conn_01x04_Pin, Connector_PinHeader_2.54mm:PinHeader_1x04_P2.54mm_Vertical, symbol Connector:Conn_01x04_Pin
- added J43: Conn_01x02_Pin, Connector_JST:JST_GH_BM02B-GHS-TBT_1x02-1MP_P1.25mm_Vertical, symbol Connector:Conn_01x02_Pin
- added R62, R63, R66, R67: 4.7k, symbol Device:R
- added R77, R79, R81, R83, R84: 10k, symbol Device:R
- added R78: 1.1k, symbol Device:R
- added R80, R82: 2.4k, symbol Device:R
- added R85: 120, symbol Device:R
- added SW1, SW2: SW_SPST, symbol Switch:SW_SPST
- added U28: TJA1462AT/0Z, SO8_SOT96-1_NXP, symbol TJA1462:TJA1462AT_0Z
- C85, C86: value C -> 10p
- renumbered D7 to D13, D7 to D3, D7 to D4, D7 to D5, D7 to D6, D7 to D8, D7 to D9, J5 to J1, J5 to J2, J5 to J3, J5 to J4, J5 to J6, J5 to J7, J5 to J8
Connections:
- net +12V: now also R79.1
- net +24V: now also R77.1
- net +3V3: now also C104.1, J23.3 (VCC), R62.1, R63.1, R66.1, R67.1, U28.5 (VIO)
- net +5V: now also C105.1, U28.3 (VCC)
- net FDCAN1_RX: now also U28.4 (RXD)
- net FDCAN1_TX: now also U28.1 (TXD)
- net I2C1_SCL: now also R63.2
- net I2C1_SDA: now also U13.140 (PB9), R62.2; no longer U13.137 (PB7)
- net I2C2_SCL: now also J33.6 (Pin_6), R66.2
- net I2C2_SDA: now also J33.5 (Pin_5), R67.2
- net NRST: now also J23.12 (~{RST})
- net SPI5_MISO: now also J33.8 (Pin_8)
- net SPI5_MOSI: now also J33.9 (Pin_9)
- net SPI5_SCK: now also J33.7 (Pin_7)
- net INA260_ALERT1: now reaches U13.1 (PE2)
- net LPUART1_TX: now reaches U13.101 (PA9)
- net LPUART1_RX: now reaches U13.102 (PA10)
- net JTMS: now reaches U13.105 (PA13(JTMS)
- net JTMS: now also J23.4 (JTMS/SWDIO)
- net at U13.106 (VCAP): now also C102.2
- net JTCK: now reaches U13.109 (PA14(JTCK)
- net JTCK: now also J23.6 (JCLK/SWCLK)
- net JTDI: now reaches U13.110 (PA15(JTDI))
- net JTDI: now also J23.10 (JTDI/NC)
- net PC12: now reaches U13.113 (PC12)
- net PC12: now also J33.4 (Pin_4)
- net PF2: now reaches U13.12 (PF2)
- net PF2: now also J42.2 (Pin_2)
- net PG10: now reaches U13.125 (PG10)
- net PG10: now also J32.1 (Pin_1)
- net PG12: now reaches U13.127 (PG12)
- net PG12: now also J32.2 (Pin_2)
- net PG13: now reaches U13.128 (PG13)
- net PG13: now also J32.3 (Pin_3)
- net PG14: now reaches U13.129 (PG14)
- net PG14: now also J32.4 (Pin_4)
- net ADC3_INP5: now reaches U13.13 (PF3)
- net ADC3_INP5: now also D30.1 (K), R79.2, R80.1
- net PG15: now reaches U13.132 (PG15)
- net PG15: now also J32.5 (Pin_5)
- net JTDO: now reaches U13.133 (PB3(JTDO)
- net JTDO: now also J23.8 (JTDO/SWO)
- net NJTRST: now reaches U13.134 (PB4(NJTRST))
- net PB5: now reaches U13.135 (PB5)
- net PB5: now also J32.6 (Pin_6)
- net PB8: now reaches U13.139 (PB8)
- net PB8: now also J32.9 (Pin_9)
- net PF4: now reaches U13.14 (PF4)
- net PF4: now also J42.3 (Pin_3)
- net FDCAN1_CTRL: now reaches U13.141 (PE0)
- net FDCAN1_CTRL: now also U28.8 (STB)
- net INA260_ALERT0: now reaches U13.142 (PE1)
- net ADC3_INP4: now reaches U13.15 (PF5)
- net ADC3_INP4: now also D29.1 (K), R77.2, R78.1
- net PF6: now reaches U13.18 (PF6)
- net PF6: now also J42.4 (Pin_4)
- net INA260_ALERT2: now reaches U13.2 (PE3)
- net ADC3_INP6: now reaches U13.22 (PF10)
- net ADC3_INP6: now also D31.1 (K), R81.2, R82.1
- net PA0: now reaches U13.34 (PA0)
- net PA0: now also J42.1 (Pin_1)
- net PF15: now reaches U13.55 (PF15)
- net PF15: now also J33.3 (Pin_3)
- net PG0: now reaches U13.56 (PG0)
- net PG0: now also J33.1 (Pin_1)
- net PG1: now reaches U13.57 (PG1)
- net PG1: now also J33.2 (Pin_2)
- net +BATT: now reaches U13.6 (VBAT)
- net +BATT: now also SW1.2 (B)
- net at U13.71 (VCAP): now also C102.1
- net PB14: now reaches U13.75 (PB14)
- net PG2: now reaches U13.87 (PG2)
- net PG2: now also J31.5 (Pin_5)
- net PG3: now reaches U13.88 (PG3)
- net PG3: now also J31.6 (Pin_6)
- net PG4: now reaches U13.89 (PG4)
- net PG4: now also J31.7 (Pin_7)
- net PG5: now reaches U13.90 (PG5)
- net PG5: now also J31.8 (Pin_8)
- net PG6: now reaches U13.91 (PG6)
- net PG6: now also J31.9 (Pin_9)
- net PG7: now reaches U13.92 (PG7)
- net PG7: now also J31.10 (Pin_10)
- net PG8: now reaches U13.93 (PG8)
- net PG8: now also J31.11 (Pin_11)
- net PC6: now reaches U13.96 (PC6)
- net PC6: now also J31.1 (Pin_1)
- net PC7: now reaches U13.97 (PC7)
- net PC7: now also J31.2 (Pin_2)
- net PC8: now reaches U13.98 (PC8)
- net PC8: now also J31.3 (Pin_3)
- net PC9: now reaches U13.99 (PC9)
- net PC9: now also J31.4 (Pin_4)
- net RTC_REFIN renamed PB15
- net PB15: now also J31.12 (Pin_12)
- new net: BT1.1 (+), SW1.1 (A)
- new net: R85.1, SW2.1 (A)
- new net: J43.2 (Pin_2), R84.2, R85.2, U28.6 (CANL)
- new net: J43.1 (Pin_1), R83.1, SW2.2 (B), U28.7 (CANH)
- new net +12L: R81.1
- new net Current Sense Block/IIN: J19.1 (Pin_1)
- new net Current Sense Block/IOUT: J19.2 (Pin_2)
- new net Current Sense Block1/IIN: J20.1 (Pin_1)
- new net Current Sense Block1/IOUT: J20.2 (Pin_2)
- new net Current Sense Block2/IIN: J21.1 (Pin_1)
- new net Current Sense Block2/IOUT: J21.2 (Pin_2)
- new net GND: BT1.2 (-), C104.2, C105.2, D29.2 (A), D30.2 (A), D31.2 (A), J23.11 (GNDDetect), J23.5 (GND), J23.7 (GND), R78.2, R80.2, R82.2, R83.2, R84.1, U28.2 (GND)
- new net Power/INPA_12V: J16.1 (Pin_1)
- new net Power/INPA_GND: J16.2 (Pin_2)
- new net Power/INPB_24V: J18.1 (Pin_1)
- new net Power/INPB_GND: J18.2 (Pin_2)
- new net USART1_RX: J32.7 (Pin_7), U13.137 (PB7)
- new net USART1_TX: J32.8 (Pin_8)
- no-connect marks 15 -> 24
Other:
- added sheet Current Sense Block (ina260sense.kicad_sch)
- added sheet Current Sense Block1 (ina260sense.kicad_sch)
- added sheet Current Sense Block2 (ina260sense.kicad_sch)
- added sheet Power (power.kicad_sch)
- note added: "A1=GND, A0=GND: Address 0b01000000 (0x40)"
- note added: "A1=GND, A0=VS: Address 0b01000001 (0x41)"
- note added: "A1=VS, A0=GND: Address 0b01000100 (0x44)"
- note added: "Exposing the unused pins on a few headers Arranged mostly based on footprint of STM32, with a few exceptions"
- note added: "External connection for the current sense Need this to use with the stepper driver, but enables us to do current sense on any other random thing if we want :)"
- note added: "JST-GH?"
- note added: "ST JTAG connector, using default KiCAD design Need to connect NJTRST somewhere or just NC?"
- note added: "STM32 H723 FT_xxx* pins can be 5.5V** tolerant, so we use a reasonable Zener. *All connected ADC pins in root sheet are FT_xxx **Actually more like 7.3V, datasheet pg 111/257"
- note added: "Should this have an opamp or buffer? Putting a zener directly on VCC seems a bit sketch lol"
- note added: "Used values from E24 resistor series for voltage divider. hopefully makes it a bit cheaper? but get like E96"
- note added: "XT60 PCB Connectors or Terminal Block (second option preferred)"
- note added: "bottom of STM32"
- note added: "left side of STM32"
- note added: "right side of STM32"
- note added: "top of STM32 used 01x12 again to keep BOM small"
- moved on the sheet: D13, D19, D20, D21, D22, D3, D4, D5, D6, D7, D8, D9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
Changed lines of the file:
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@@
-(kicad_sch (version 20230121) (generator eeschema)
-  (paper "A2")
+(kicad_sch
+	(version 20231120)
+	(generator "eeschema")
+	(generator_version "8.0")
+	(paper "A1")

Commit message: added footprints to almost all components
Parts:
- removed J1, J2, J3, J4, J5, J6, J7, J8: Screw_Terminal_01x02, symbol Connector:Screw_Terminal_01x02
- removed J16, J18, J19, J20, J21: Conn_01x02_Socket, symbol Connector:Conn_01x02_Socket
- removed J31, J32, J33: Conn_01x12_Pin, Connector_PinHeader_2.54mm:PinHeader_1x12_P2.54mm_Vertical, symbol Connector:Conn_01x12_Pin
- removed J42: Conn_01x04_Pin, Connector_PinHeader_2.54mm:PinHeader_1x04_P2.54mm_Vertical, symbol Connector:Conn_01x04_Pin
- removed J43: Conn_01x02_Pin, Connector_JST:JST_GH_BM02B-GHS-TBT_1x02-1MP_P1.25mm_Vertical, symbol Connector:Conn_01x02_Pin
- removed SW1, SW2: SW_SPST, symbol Switch:SW_SPST
- added C106, C107, C108, C109, C110, C111, C113, C114, C115, C116, C117, C118: 100n, Capacitor_SMD:C_0603_1608Metric_Pad1.08x0.95mm_HandSolder, symbol Device:C_Small
- added C112, C121: 1u, Capacitor_SMD:C_0603_1608Metric_Pad1.08x0.95mm_HandSolder, symbol Device:C_Small
- added C119: 4.7u, Capacitor_SMD:C_0603_1608Metric_Pad1.08x0.95mm_HandSolder, symbol Device:C
- added C120: 2.2u, Capacitor_SMD:C_0603_1608Metric_Pad1.08x0.95mm_HandSolder, symbol Device:C
- added C125, C126: 100n, Capacitor_SMD:C_0603_1608Metric_Pad1.08x0.95mm_HandSolder, symbol Device:C
- added FB1: FerriteBead, Inductor_SMD:L_0805_2012Metric_Pad1.15x1.40mm_HandSolder, symbol Device:FerriteBead
- added J1, J10, J12, J13, J2, J3, J4, J5, J6, J7, J8: Conn_01x04, Connector_Phoenix_MSTB:PhoenixContact_MSTBA_2,5_4-G-5,08_1x04_P5.08mm_Horizontal, symbol Connector_Generic:Conn_01x04
- added J15, J9: Conn_01x04, Connector_JST:JST_GH_BM04B-GHS-TBT_1x04-1MP_P1.25mm_Vertical, symbol Connector_Generic:Conn_01x04
- added J16, J18: Conn_01x02, Connector_Phoenix_MSTB:PhoenixContact_MSTBA_2,5_2-G-5,08_1x02_P5.08mm_Horizontal, symbol Connector_Generic:Conn_01x02
- added J19, J20, J21, J32: Conn_01x02, Connector_PinHeader_2.54mm:PinHeader_1x02_P2.54mm_Vertical, symbol Connector_Generic:Conn_01x02
- added J38: Conn_01x12, Connector_PinHeader_2.54mm:PinHeader_1x12_P2.54mm_Vertical, symbol Connector_Generic:Conn_01x12
- added U30, U31, U32: Pololu 36v4 Breakout, symbol LaunchpadControllerLib:Pololu_36v4
- added U33: TJA1462AT/0Z, SO8_SOT96-1_NXP, symbol TJA1462:TJA1462AT_0Z
- BT1: footprint Battery:Battery_Panasonic_CR2032-VS1N_Vertical_CircularHoles -> Battery:BatteryHolder_Keystone_1057_1x2032; Mouser# (none) -> 534-1057
- C102: value 22u -> 2.2u; footprint (none) -> Capacitor_SMD:C_0603_1608Metric_Pad1.08x0.95mm_HandSolder
- C104, C105, C83, C84, C85, C86: footprint (none) -> Capacitor_SMD:C_0603_1608Metric_Pad1.08x0.95mm_HandSolder
- D13, D3, D4, D5, D6, D7, D8, D9: footprint (none) -> Diode_SMD:D_0805_2012Metric_Pad1.15x1.40mm_HandSolder; Mouser# (none) -> 821-BZY55C33RBG
- D19, D20, D21, D22: footprint (none) -> LED_SMD:LED_0805_2012Metric_Pad1.15x1.40mm_HandSolder
- D29, D30, D31: footprint (none) -> Package_TO_SOT_SMD:SOT-23_Handsoldering; Mouser# (none) -> 771-PLVA650A-QR
- R22, R23, R24, R25, R27, R28, R29, R31, R34, R35, R38, R39, R42, R43, R44, R45, R62, R63, R66, R67, R77, R78, R79, R80, R81, R82, R83, R85: footprint (none) -> Resistor_SMD:R_0805_2012Metric_Pad1.20x1.40mm_HandSolder
- R54, R55, R56, R57: value 250 -> 500; footprint (none) -> Resistor_SMD:R_0805_2012Metric_Pad1.20x1.40mm_HandSolder
- R84: value 10k -> 120; footprint (none) -> Resistor_SMD:R_0805_2012Metric_Pad1.20x1.40mm_HandSolder
- U21, U22: footprint (none) -> Package_SO:SOIC-14_3.9x8.7mm_P1.27mm; Mouser# (none) -> 595-SN74LS06NSRG4
Connections:
- net BOOT0 is gone; now on net GND: U13.138 (BOOT0)
- net GNDA is gone; now on net GND: C83.2, C84.2, C85.2, C86.2, U13.31 (VSSA), Y1.2
- net GNDD is gone; now on net GND: D13.2 (A), D3.2 (A), D4.2 (A), D5.2 (A), D6.2 (A), D7.2 (A), D8.2 (A), D9.2 (A), R29.2, R31.2, R35.2, R39.2, R42.2, R43.2, R44.2, R45.2, U13.107 (VSS), U13.120 (VSS), U13.130 (VSS), U13.16 (VSS), U13.38 (VSS), U13.51 (VSS), U13.61 (VSS), U13.83 (VSS), U13.94 (VSS), U21.7 (GND), U22.7 (GND)
- net PG0 is gone; now on net MOTOR1_nFAULT: U13.56 (PG0)
- net PG1 is gone; now on net MOTOR1_nSTALL: U13.57 (PG1)
- net PG12 is gone; now on net ETH_TXD0: U13.127 (PG12)
- net PG13 is gone; now on net ETH_TXD1: U13.128 (PG13)
- net PG2 is gone; now on net MOTOR2_nFAULT: U13.87 (PG2)
- net PG3 is gone; now on net MOTOR2_nSTALL: U13.88 (PG3)
- net PG4 is gone; now on net MOTOR3_nFAULT: U13.89 (PG4)
- net PG5 is gone; now on net MOTOR3_nSTALL: U13.90 (PG5)
- net VREFBUF_OUT is gone; now on net +3V3: U13.32 (VREF+)
- net +12V: now also J15.1 (Pin_1), J9.1 (Pin_1)
- net +3V3: now also R83.2, U13.143 (PDR_ON), C106.1, C107.1, C108.1, C109.1, C110.1, C112.1, C113.1, C114.1, C115.1, C116.1, C117.1, C118.1, C119.1, C126.1, FB1.2, U30.10 (nSLP), U30.2 (IOREF), U31.10 (nSLP), U31.2 (IOREF), U32.10 (nSLP), U32.2 (IOREF), U33.5 (VIO); no longer U13.33 (VDDA)
- net +5V: now also C125.1, U33.3 (VCC)
- net +BATT: now also J20.2 (Pin_2)
- net High Side Switch/OUT: now also J5.2 (Pin_2)
- net ADC1_INP2: now also U32.16 (BEMF)
- net ADC1_INP3: now also U31.16 (BEMF)
- net ADC1_INP5: now also U30.16 (BEMF)
- net Current Sense Block/IOUT: now also U32.17 (VIN), U32.18 (VIN)
- net Current Sense Block1/IOUT: now also U30.17 (VIN), U30.18 (VIN)
- net Current Sense Block2/IOUT: now also U31.17 (VIN), U31.18 (VIN)
- net ETH_TXD0: no longer U13.73 (PB12)
- net ETH_TXD1: no longer U13.74 (PB13)
- net GND: now also C102.2, C106.2, C107.2, C108.2, C109.2, C110.2, C111.2, C112.2, C113.2, C114.2, C115.2, C116.2, C117.2, C118.2, C119.2, C120.2, C121.2, C125.2, C126.2, J1.3 (Pin_3), J1.4 (Pin_4), J15.4 (Pin_4), J19.2 (Pin_2), J2.3 (Pin_3), J2.4 (Pin_4), J3.3 (Pin_3), J3.4 (Pin_4), J4.3 (Pin_3), J4.4 (Pin_4), J5.3 (Pin_3), J5.4 (Pin_4), J6.3 (Pin_3), J6.4 (Pin_4), J7.3 (Pin_3), J7.4 (Pin_4), J8.3 (Pin_3), J8.4 (Pin_4), J9.4 (Pin_4), U30.19 (GND), U30.20 (GND), U30.3 (IOGND), U31.19 (GND), U31.20 (GND), U31.3 (IOGND), U32.19 (GND), U32.20 (GND), U32.3 (IOGND), U33.2 (GND); no longer R83.2, R84.1
- net I2C2_SCL: now also J38.2 (Pin_2)
- net I2C2_SDA: now also J38.1 (Pin_1)
- net MOTOR1_DIR: now also U31.5 (DIR)
- net MOTOR1_SCS: now also U31.9 (SCS)
- net MOTOR1_STEP: now also U31.4 (STEP)
- net MOTOR1_nFAULT: now also U31.12 (nFLT)
- net MOTOR1_nSTALL: now also U31.15 (nSTALL)
- net MOTOR2_DIR: now also U32.5 (DIR)
- net MOTOR2_SCS: now also U32.9 (SCS)
- net MOTOR2_STEP: now also U32.4 (STEP)
- net MOTOR2_nFAULT: now also U32.12 (nFLT)
- net MOTOR2_nSTALL: now also U32.15 (nSTALL)
- net MOTOR3_DIR: now also U30.5 (DIR)
- net MOTOR3_SCS: now also U30.9 (SCS)
- net MOTOR3_STEP: now also U30.4 (STEP)
- net MOTOR3_nFAULT: now also U30.12 (nFLT)
- net MOTOR3_nSTALL: now also U30.15 (nSTALL)
- net PF6: now also J38.12 (Pin_12)
- net PG14: now also J38.10 (Pin_10)
- net PG15: now also J38.11 (Pin_11)
- net PG7: now also J38.8 (Pin_8)
- net PG8: now also J38.9 (Pin_9)
- net Power/INPA_12V: now also J16.1 (Pin_1)
- net Power/INPA_GND: now also J16.2 (Pin_2)
- net Power/INPB_24V: now also J18.1 (Pin_1)
- net Power/INPB_GND: now also J18.2 (Pin_2)
- net SPI3_MISO: now also U30.6 (SDATO), U31.7 (SDATI), U32.7 (SDATI)
- net SPI3_MOSI: now also U30.7 (SDATI), U31.6 (SDATO), U32.6 (SDATO)
- net SPI3_SCK: now also U30.8 (SCLK), U31.8 (SCLK), U32.8 (SCLK)
- net SPI5_MISO: now also J38.4 (Pin_4)
- net SPI5_MOSI: now also J38.5 (Pin_5)
- net SPI5_SCK: now also J38.3 (Pin_3)
- net USART1_RX: now also J38.6 (Pin_6)
- net USART1_TX: now also J38.7 (Pin_7)
- net at BT1.1 (+): now also J20.1 (Pin_1)
- net at R85.1: now also J21.2 (Pin_2)
- net at R85.2, U28.6 (CANL): now also J15.3 (Pin_3); no longer R84.2
- net at R83.1: now also J19.1 (Pin_1); no longer U28.7 (CANH)
- net at U13.106 (VCAP): now also C120.1; no longer C102.2
- net 12V High Side Switch/IN renamed High Side Switch4/IN
- net 12V High Side Switch/OUT renamed High Side Switch4/OUT
- net High Side Switch4/OUT: now also J1.2 (Pin_2)
- net 12V High Side Switch1/IN renamed High Side Switch5/IN
- net 12V High Side Switch1/OUT renamed High Side Switch5/OUT
- net High Side Switch5/OUT: now also J2.2 (Pin_2)
- net 12V High Side Switch2/IN renamed High Side Switch6/IN
- net 12V High Side Switch2/OUT renamed High Side Switch6/OUT
- net High Side Switch6/OUT: now also J3.2 (Pin_2)
- net 12V High Side Switch3/IN renamed High Side Switch7/IN
- net 12V High Side Switch3/OUT renamed High Side Switch7/OUT
- net High Side Switch7/OUT: now also J4.2 (Pin_2)
- net 24V High Side Switch1/IN renamed High Side Switch1/IN
- net 24V High Side Switch1/OUT renamed High Side Switch1/OUT
- net High Side Switch1/OUT: now also J6.2 (Pin_2)
- net 24V High Side Switch2/IN renamed High Side Switch2/IN
- net 24V High Side Switch2/OUT renamed High Side Switch2/OUT
- net High Side Switch2/OUT: now also J7.2 (Pin_2)
- net 24V High Side Switch3/IN renamed High Side Switch3/IN
- net 24V High Side Switch3/OUT renamed High Side Switch3/OUT
- net High Side Switch3/OUT: now also J8.2 (Pin_2)
- net PA0: no longer names the net of U13.34 (PA0)
- net PB14 renamed FDCAN2_CTRL
- net FDCAN2_CTRL: now also U33.8 (STB)
- net PB15: no longer names the net of U13.76 (PB15)
- net PB5: no longer names the net of U13.135 (PB5)
- net PB8: no longer names the net of U13.139 (PB8)
- net PC12: no longer names the net of U13.113 (PC12)
- net PC6: no longer names the net of U13.96 (PC6)
- net PC7: no longer names the net of U13.97 (PC7)
- net PC8: no longer names the net of U13.98 (PC8)
- net PC9: no longer names the net of U13.99 (PC9)
- net PF15: no longer names the net of U13.55 (PF15)
- net PF2: no longer names the net of U13.12 (PF2)
- net PF4: no longer names the net of U13.14 (PF4)
- net PG10: no longer names the net of U13.125 (PG10)
- net PG6: no longer names the net of U13.91 (PG6)
- new net: J10.1 (Pin_1), U30.21 (AOUT1)
- new net: J10.2 (Pin_2), U30.22 (AOUT2)
- new net: J10.3 (Pin_3), U30.23 (BOUT1)
- new net: J10.4 (Pin_4), U30.24 (BOUT2)
- new net: J12.1 (Pin_1), U32.21 (AOUT1)
- new net: J12.2 (Pin_2), U32.22 (AOUT2)
- new net: J12.3 (Pin_3), U32.23 (BOUT1)
- new net: J12.4 (Pin_4), U32.24 (BOUT2)
- new net: J13.1 (Pin_1), U31.21 (AOUT1)
- new net: J13.2 (Pin_2), U31.22 (AOUT2)
- new net: J13.3 (Pin_3), U31.23 (BOUT1)
- new net: J13.4 (Pin_4), U31.24 (BOUT2)
- new net: C111.1, C121.1, FB1.1, U13.33 (VDDA)
- new net: J9.3 (Pin_3), R84.2, U33.6 (CANL)
- new net: J32.1 (Pin_1), J9.2 (Pin_2), U33.7 (CANH)
- new net: J15.2 (Pin_2), J21.1 (Pin_1), U28.7 (CANH)
- new net: J32.2 (Pin_2), R84.1
- new net FDCAN2_RX: U13.73 (PB12), U33.4 (RXD)
- new net FDCAN2_TX: U13.74 (PB13), U33.1 (TXD)
- new net High Side Switch/Vbb: J5.1 (Pin_1)
- new net High Side Switch1/Vbb: J6.1 (Pin_1)
- new net High Side Switch2/Vbb: J7.1 (Pin_1)
- new net High Side Switch3/Vbb: J8.1 (Pin_1)
- new net High Side Switch4/Vbb: J1.1 (Pin_1)
- new net High Side Switch5/Vbb: J2.1 (Pin_1)
- new net High Side Switch6/Vbb: J3.1 (Pin_1)
- new net High Side Switch7/Vbb: J4.1 (Pin_1)
- no-connect marks 24 -> 38
Other:
- sheet 24V High Side Switch renamed High Side Switch
- removed sheet 12V High Side Switch
- removed sheet 12V High Side Switch1
- removed sheet 12V High Side Switch2
- removed sheet 12V High Side Switch3
- removed sheet 24V High Side Switch1
- removed sheet 24V High Side Switch2
- removed sheet 24V High Side Switch3
- removed sheet Pololu Stepper Motor Driver 36v4 Breakout
- removed sheet Pololu Stepper Motor Driver 36v4 Breakout1
- removed sheet Pololu Stepper Motor Driver 36v4 Breakout2
- added sheet High Side Switch1 (hss.kicad_sch)
- added sheet High Side Switch2 (hss.kicad_sch)
- added sheet High Side Switch3 (hss.kicad_sch)
- added sheet High Side Switch4 (hss.kicad_sch)
- added sheet High Side Switch5 (hss.kicad_sch)
- added sheet High Side Switch6 (hss.kicad_sch)
- added sheet High Side Switch7 (hss.kicad_sch)
- sheet ADC1 ports: added none; removed REFOUT
- sheet ADC2 ports: added none; removed REFOUT
- note added: "Add decoupling caps on each pin, and a big one on the supply"
- note added: "Add decoupling caps on each pin, and a big one on the supply 100n"
- note added: "Exposing some useful pins"
- note added: "JST-GH"
- note added: "PDR_ON HIGH => enable power supply supervisor"
- note added: "TODO: Check with Fjalar schematic (pull up or pull down)?"
- note added: "Tie GND, GNDA, and GNDD"
- note removed: "Exposing the unused pins on a few headers Arranged mostly based on footprint of STM32, with a few exceptions"
- note removed: "External connection for the current sense Need this to use with the stepper driver, but enables us to do current sense on any other random thing if we want :)"
- note removed: "JST-GH?"
- note removed: "bottom of STM32"
- note removed: "left side of STM32"
- note removed: "right side of STM32"
- note removed: "top of STM32 used 01x12 again to keep BOM small"
- moved on the sheet: C102, C104, C105, D19, D20, D21, D22, D7, R22, R23, R24, R25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
