File: launchpad-controller-v2.kicad_sch (KiCad schematic)
At the start: 78 parts, among them J10 Conn_01x04, J12 Conn_01x04, J13 Conn_01x04, J15 Conn_01x04, J16 Conn_01x02, J18 Conn_01x02, J19 Conn_01x02, J21 Conn_01x02, J23 Conn_ST_STDC14, J32 Conn_01x02, J38 Conn_01x12, J9 Conn_01x04, U13 STM32H723ZGTx, U21 74LS06, U22 74LS06, U28 TJA1462AT/0Z, U30 Pololu 36v4 Breakout, U31 Pololu 36v4 Breakout, U32 Pololu 36v4 Breakout, U33 TJA1462AT/0Z, Y1 50MHz

Commit message: routing done
Parts:
- removed D31: 5V, Package_TO_SOT_SMD:SOT-23_Handsoldering, symbol Device:D_Zener
- removed J38: Conn_01x12, Connector_PinHeader_2.54mm:PinHeader_1x12_P2.54mm_Vertical, symbol Connector_Generic:Conn_01x12
- removed R66, R67: 4.7k, Resistor_SMD:R_0603_1608Metric_Pad0.98x0.95mm_HandSolder, symbol Device:R
- removed R81: 10k, Resistor_SMD:R_0603_1608Metric_Pad0.98x0.95mm_HandSolder, symbol Device:R
- removed R82: 2.4k, Resistor_SMD:R_0603_1608Metric_Pad0.98x0.95mm_HandSolder, symbol Device:R
Connections:
- net +BATT is gone; now on net +3V3: U13.6 (VBAT)
- net ADC1_ERROR is gone; now on net SW5_IN: U13.5 (PE6)
- net I2C2_SCL is gone; now on net nLED24_2: U13.11 (PF1)
- net I2C2_SDA is gone; now on net nLED24_1: U13.10 (PF0)
- net PG14 is gone; now on net MOTOR3_nFAULT: U13.129 (PG14)
- net PG15 is gone; now on net MOTOR3_nSTALL: U13.132 (PG15)
- net USART1_RX is gone; now on net I2C1_SDA: U13.137 (PB7)
- net USART1_TX is gone; now on net nLED12_1: U13.75 (PB14)
- net ADC1_CS: now also U13.1 (PE2); no longer U13.64 (PE11)
- net ADC1_SYNC: now also U13.2 (PE3); no longer U13.3 (PE4)
- net ADC2_CS: now also U13.3 (PE4); no longer U13.65 (PE12)
- net FDCAN1_RX: now also U13.139 (PB8), U33.4 (RXD); no longer U13.103 (PA11), U28.4 (RXD)
- net FDCAN1_TX: now also U13.140 (PB9), U33.1 (TXD); no longer U13.104 (PA12), U28.1 (TXD)
- net I2C1_SDA: no longer U13.140 (PB9)
- net MOTOR1_DIR: now also U13.91 (PG6); no longer U13.116 (PD2)
- net MOTOR1_SCS: now also U13.114 (PD0); no longer U13.59 (PE8)
- net MOTOR1_STEP: now also U13.90 (PG5); no longer U13.115 (PD1)
- net MOTOR1_nFAULT: now also U13.115 (PD1), U31.12 (nFLT); no longer U13.56 (PG0)
- net MOTOR1_nSTALL: now also U13.116 (PD2); no longer U13.57 (PG1)
- net MOTOR2_DIR: now also U13.86 (PD15); no longer U13.118 (PD4)
- net MOTOR2_SCS: now also U13.87 (PG2); no longer U13.60 (PE9)
- net MOTOR2_STEP: now also U13.85 (PD14); no longer U13.117 (PD3)
- net MOTOR2_nFAULT: now also U13.88 (PG3); no longer U13.87 (PG2)
- net MOTOR2_nSTALL: now also U13.89 (PG4); no longer U13.88 (PG3)
- net MOTOR3_DIR: now also U13.118 (PD4); no longer U13.122 (PD6)
- net MOTOR3_SCS: now also U13.119 (PD5); no longer U13.63 (PE10)
- net MOTOR3_STEP: now also U13.117 (PD3); no longer U13.119 (PD5)
- net MOTOR3_nFAULT: no longer U13.89 (PG4)
- net MOTOR3_nSTALL: no longer U13.90 (PG5)
- net SPI3_MOSI: now also U13.113 (PC12); no longer U13.48 (PB2)
- net SW5_IN: no longer U13.81 (PD12)
- net SW6_IN: now also U13.7 (PC13); no longer U13.82 (PD13)
- net SW7_IN: now also U13.8 (PC14); no longer U13.85 (PD14)
- net SW8_IN: now also U13.9 (PC15); no longer U13.86 (PD15)
- net nLED12_1: no longer U13.114 (PD0)
- net nLED12_2: now also U13.74 (PB13); no longer U13.66 (PE13)
- net nLED24_1: no longer U13.67 (PE14)
- net nLED24_2: no longer U13.68 (PE15)
- net ADC1_INP2 renamed 12_VSENSE
- net 12_VSENSE: now also D30.1 (K), R79.2, R80.1; no longer U32.16 (BEMF)
- net ADC1_INP3 renamed MOTOR1_BEMF
- net MOTOR1_BEMF: now also U13.13 (PF3); no longer U13.42 (PA6)
- net ADC1_INP5 renamed MOTOR3_BEMF
- net ADC1_INP6 renamed 24_VSENSE
- net 24_VSENSE: now also D29.1 (K), R77.2, R78.1
- net ADC2_ERROR: no longer names the net of U13.58 (PE7)
- net ADC2_INP10 renamed SW4_ADC
- net ADC2_INP15 renamed SW5_ADC
- net ADC2_INP18 renamed SW6_ADC
- net ADC2_INP19 renamed SW7_ADC
- net ADC2_INP2 renamed SW1_ADC
- net ADC2_INP6 renamed SW2_ADC
- net ADC2_INP9 renamed SW3_ADC
- removed net ADC3_INP4: D29.1 (K), R77.2, R78.1, U13.15 (PF5)
- removed net ADC3_INP5: D30.1 (K), R79.2, R80.1, U13.13 (PF3)
- net FDCAN2_RX: no longer names the net of U13.73 (PB12)
- net FDCAN2_RX: no longer U33.4 (RXD)
- removed net FDCAN2_TX: U13.74 (PB13), U33.1 (TXD)
- net LPUART1_RX: no longer names the net of U13.102 (PA10)
- net LPUART1_TX: no longer names the net of U13.101 (PA9)
- net PF6 renamed FDCAN3_RX
- net FDCAN3_RX: now also U28.4 (RXD)
- net PG7: no longer names the net of U13.92 (PG7)
- net PG8: no longer names the net of U13.93 (PG8)
- net SPI5_MISO: no longer names the net of U13.20 (PF8)
- net SPI5_MOSI: no longer names the net of U13.21 (PF9)
- net SPI5_SCK renamed FDCAN3_TX
- net FDCAN3_TX: now also U28.1 (TXD)
- new net MOTOR2_BEMF: U13.42 (PA6), U32.16 (BEMF)
- new net SW8_ADC: U13.15 (PF5)
- no-connect marks 50 -> 55
Other:
- note removed: "Exposing some useful pins"
- moved on the sheet: R62
