File: launchpad-controller-v2.kicad_sch (KiCad schematic)
At the start: 72 parts, among them J10 Conn_01x04, J12 Conn_01x04, J13 Conn_01x04, J15 Conn_01x04, J16 Conn_01x02, J18 Conn_01x02, J19 Conn_01x02, J21 Conn_01x02, J23 Conn_ST_STDC14, J32 Conn_01x02, J9 Conn_01x04, U13 STM32H723ZGTx, U21 74LS06, U22 74LS06, U28 TJA1462AT/0Z, U30 Pololu 36v4 Breakout, U31 Pololu 36v4 Breakout, U32 Pololu 36v4 Breakout, U33 TJA1462AT/0Z, Y1 50MHz

Commit message: bajs
Parts:
- renumbered C105 to C57, C104 to C58, C125 to C59, C126 to C60, C102 to C68, C117 to C69, C110 to C70, C118 to C71, C119 to C72, C120 to C73, C116 to C74, C112 to C75, C115 to C76, C109 to C77, C114 to C78, C106 to C79, C108 to C80, C107 to C81, C111 to C82, C121 to C83, C113 to C85, C83 to C86, D19 to D11, D20 to D19, D21 to D23, D30 to D5, D29 to D7, FB1 to FB2, H3 to H2, H2 to H3, J16 to J1, J12 to J15, J18 to J2, J13 to J24, J21 to J27, J10 to J28, J15 to J29, J9 to J30, J32 to J31, J23 to J7, J19 to J8, R105 to R1, R80 to R12, R79 to R13, R77 to R15, R78 to R16, R54 to R20, R106 to R31, R83 to R32, R55 to R33, R63 to R34, R62 to R35, R56 to R62, R57 to R63, R85 to R64, R104 to R65, R103 to R8, R102 to R86, R84 to R87, U31 to U12, U30 to U23, U28 to U24, U33 to U25, U21 to U28, U13 to U33, U22 to U6, U32 to U9
Connections:
- net ADC3_INP6: no longer names the net of U33.22 (PF10)
- net NJTRST: no longer names the net of U33.134 (PB4(NJTRST))
- no-connect marks 55 -> 60

Commit message: bajs
Parts:
- added H5, H6: MountingHole_Pad, MountingHole:MountingHole_4.3mm_M4_Pad_Via, symbol Mechanical:MountingHole_Pad
- added R103, R104: 100k, Resistor_SMD:R_0603_1608Metric_Pad0.98x0.95mm_HandSolder, symbol Device:R
Connections:
- net Earth: now also R103.2, R104.2
- net SPI3_MISO: now also U12.6 (SDATO), U9.6 (SDATO); no longer U12.7 (SDATI), U9.7 (SDATI)
- net SPI3_MOSI: now also U12.7 (SDATI), U9.7 (SDATI); no longer U12.6 (SDATO), U9.6 (SDATO)
- new net: H6.1, R104.1
- new net: H5.1, R103.1
