File: pololu_36v4_breakout.kicad_sch (KiCad schematic)
At the start: 2 parts, among them J10 Conn_01x04_Socket, J9 Conn_01x12_Socket

Commit message: Launchpad controller revision 06/03/2024
Parts:
- J10: footprint Connector:FanPinHeader_1x04_P2.54mm_Vertical -> Connector_PinSocket_2.54mm:PinSocket_1x04_P2.54mm_Vertical
- J9: footprint (none) -> Connector_PinSocket_2.54mm:PinSocket_1x12_P2.54mm_Vertical
Other:
- note added: "Careful when routing. Try to keep the spacing the same as the Pololu 36v4 Driver"
- moved on the sheet: J10, J9
