File: ethphy.kicad_sch (KiCad schematic)
At the start: 21 parts, among them J11 ARJM11A1-009-AB-EW2, U2 DP83848KSQ/NOPB

Commit message: bajs
Parts:
- renumbered C88 to C1, C79 to C2, C87 to C3, C1 to C61, C80 to C62, C89 to C63, C5 to C64, C90 to C65, C82 to C66, C81 to C67, J11 to J6, R21 to R10, R18 to R88, R17 to R89, R20 to R9, R19 to R90, R61 to R91, R60 to R92, R59 to R93, R58 to R94, U2 to U32
Connections:
- net GNDA: now also U32.41 (EPAD)
- no-connect marks 14 -> 13
Changed lines of the file:
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@@
 	)
 	(junction
+		(at 144.78 90.17)
+		(diameter 0)
+		(color 0 0 0 0)
+	)
+	(junction
 		(at 220.98 44.45)
 		(diameter 0)
@@
 	)
 	(no_connect
-		(at 139.7 85.09)
-	)
-	(no_connect
 		(at 63.5 52.07)
 	)
@@
 	(wire
 		(pts
+			(xy 144.78 90.17) (xy 153.67 90.17)
+		)
+		(stroke
+			(width 0)
+			(type default)
+		)
+	)
+	(wire
+		(pts
 			(xy 34.29 87.63) (xy 63.5 87.63)
 		)
@@
 	(wire
 		(pts
-			(xy 139.7 90.17) (xy 153.67 90.17)
+			(xy 139.7 90.17) (xy 144.78 90.17)
 		)
 		(stroke
@@
 	(wire
 		(pts
+			(xy 139.7 85.09) (xy 144.78 85.09)
+		)
+		(stroke
+			(width 0)
+			(type default)
+		)
+	)
+	(wire
+		(pts
 			(xy 120.65 152.4) (xy 140.97 152.4)
 		)
@@
 	(wire
 		(pts
+			(xy 144.78 85.09) (xy 144.78 90.17)
+		)
+		(stroke
+			(width 0)
+			(type default)
+		)
+	)
+	(wire
+		(pts
 			(xy 31.75 54.61) (xy 29.21 54.61)
 		)
@@
 		(dnp no)
 		(fields_autoplaced yes)
-		(property "Reference" "C5"
+		(property "Reference" "C64"
 			(at 58.42 107.9499 0)
 			(effects
@@
 			(project "launchpad-controller-v2"
 				(path "/8b86c7a7-6364-4b1f-ab12-b4882a7d8ae2/8c27322b-4514-4c93-94e3-74166c34f228"
-					(reference "C5")
+					(reference "C64")
 					(unit 1)
 				)
@@
 		(on_board yes)
 		(dnp no)
-		(property "Reference" "C82"
+		(property "Reference" "C66"
 			(at 175.26 82.55 0)
 			(effects
@@
 			(project "launchpad-controller-v2"
 				(path "/8b86c7a7-6364-4b1f-ab12-b4882a7d8ae2/8c27322b-4514-4c93-94e3-74166c34f228"
-					(reference "C82")
+					(reference "C66")
 					(unit 1)
 				)
@@
 		(on_board yes)
 		(dnp no)
-		(property "Reference" "C81"
+		(property "Reference" "C67"
 			(at 163.83 82.55 0)
 			(effects
@@
 			(project "launchpad-controller-v2"
 				(path "/8b86c7a7-6364-4b1f-ab12-b4882a7d8ae2/8c27322b-4514-4c93-94e3-74166c34f228"
-					(reference "C81")
+					(reference "C67")
 					(unit 1)
 				)
@@
 		(dnp no)
 		(fields_autoplaced yes)
-		(property "Reference" "C90"
+		(property "Reference" "C65"
 			(at 46.99 154.94 0)
 			(effects
@@
 			(project "launchpad-controller-v2"
 				(path "/8b86c7a7-6364-4b1f-ab12-b4882a7d8ae2/8c27322b-4514-4c93-94e3-74166c34f228"
-					(reference "C90")
+					(reference "C65")
 					(unit 1)
 				)
@@
 		(dnp no)
 		(fields_autoplaced yes)
-		(property "Reference" "R17"
+		(property "Reference" "R89"
 			(at 36.83 31.75 0)
 			(effects
@@
 			(project "launchpad-controller-v2"
 				(path "/8b86c7a7-6364-4b1f-ab12-b4882a7d8ae2/8c27322b-4514-4c93-94e3-74166c34f228"
-					(reference "R17")
+					(reference "R89")
 					(unit 1)
 				)
@@
 		(dnp no)
 		(fields_autoplaced yes)
-		(property "Reference" "C89"
+		(property "Reference" "C63"
 			(at 34.29 152.4 0)
 			(effects
@@
 			(project "launchpad-controller-v2"
 				(path "/8b86c7a7-6364-4b1f-ab12-b4882a7d8ae2/8c27322b-4514-4c93-94e3-74166c34f228"
-					(reference "C89")
+					(reference "C63")
 					(unit 1)
 				)
@@
 		(dnp no)
 		(fields_autoplaced yes)
-		(property "Reference" "R60"
+		(property "Reference" "R92"
 			(at 222.25 74.93 0)
 			(effects
@@
 			(project "launchpad-controller-v2"
 				(path "/8b86c7a7-6364-4b1f-ab12-b4882a7d8ae2/8c27322b-4514-4c93-94e3-74166c34f228"
-					(reference "R60")
+					(reference "R92")
 					(unit 1)
 				)
@@
 		(on_board yes)
 		(dnp no)
-		(property "Reference" "R18"
+		(property "Reference" "R88"
 			(at 35.56 48.26 90)
 			(effects
@@
 			(project "launchpad-controller-v2"
 				(path "/8b86c7a7-6364-4b1f-ab12-b4882a7d8ae2/8c27322b-4514-4c93-94e3-74166c34f228"
-					(reference "R18")
+					(reference "R88")
 					(unit 1)
 				)
@@
 		(dnp no)
 		(fields_autoplaced yes)
-		(property "Reference" "J11"
+		(property "Reference" "J6"
 			(at 97.79 132.08 0)
 			(effects
@@
 			(project "launchpad-controller-v2"
 				(path "/8b86c7a7-6364-4b1f-ab12-b4882a7d8ae2/8c27322b-4514-4c93-94e3-74166c34f228"
-					(reference "J11")
+					(reference "J6")
 					(unit 1)
 				)
@@
 		(dnp no)
 		(fields_autoplaced yes)
-		(property "Reference" "C79"
+		(property "Reference" "C2"
 			(at 26.67 87.63 0)
 			(effects
@@
 			(project "launchpad-controller-v2"
 				(path "/8b86c7a7-6364-4b1f-ab12-b4882a7d8ae2/8c27322b-4514-4c93-94e3-74166c34f228"
-					(reference "C79")
+					(reference "C2")
 					(unit 1)
 				)
@@
 		(dnp no)
 		(fields_autoplaced yes)
-		(property "Reference" "R21"
+		(property "Reference" "R10"
 			(at 152.4 148.59 90)
 			(effects
@@
 			(project "launchpad-controller-v2"
 				(path "/8b86c7a7-6364-4b1f-ab12-b4882a7d8ae2/8c27322b-4514-4c93-94e3-74166c34f228"
-					(reference "R21")
+					(reference "R10")
 					(unit 1)
 				)
@@
 		(dnp no)
 		(fields_autoplaced yes)
-		(property "Reference" "C87"
+		(property "Reference" "C3"
 			(at 241.3 46.99 0)
 			(effects
@@
 			(project "launchpad-controller-v2"
 				(path "/8b86c7a7-6364-4b1f-ab12-b4882a7d8ae2/8c27322b-4514-4c93-94e3-74166c34f228"
-					(reference "C87")
+					(reference "C3")
 					(unit 1)
 				)
@@
 		(on_board yes)
 		(dnp no)
-		(property "Reference" "C80"
+		(property "Reference" "C62"
 			(at 38.1 90.17 0)
 			(effects
@@
 			(project "launchpad-controller-v2"
 				(path "/8b86c7a7-6364-4b1f-ab12-b4882a7d8ae2/8c27322b-4514-4c93-94e3-74166c34f228"
-					(reference "C80")
+					(reference "C62")
 					(unit 1)
 				)
@@
 		(dnp no)
 		(fields_autoplaced yes)
-		(property "Reference" "C1"
+		(property "Reference" "C61"
 			(at 45.72 107.95 0)
 			(effects
@@
 			(project "launchpad-controller-v2"
 				(path "/8b86c7a7-6364-4b1f-ab12-b4882a7d8ae2/8c27322b-4514-4c93-94e3-74166c34f228"
-					(reference "C1")
+					(reference "C61")
 					(unit 1)
 				)
@@
 		(dnp no)
 		(fields_autoplaced yes)
-		(property "Reference" "R20"
+		(property "Reference" "R9"
 			(at 152.4 138.43 90)
 			(effects
@@
 			(project "launchpad-controller-v2"
 				(path "/8b86c7a7-6364-4b1f-ab12-b4882a7d8ae2/8c27322b-4514-4c93-94e3-74166c34f228"
-					(reference "R20")
+					(reference "R9")
 					(unit 1)
 				)
@@
 		(dnp no)
 		(fields_autoplaced yes)
-		(property "Reference" "R59"
+		(property "Reference" "R93"
 			(at 223.52 50.8 0)
 			(effects
@@
 			(project "launchpad-controller-v2"
 				(path "/8b86c7a7-6364-4b1f-ab12-b4882a7d8ae2/8c27322b-4514-4c93-94e3-74166c34f228"
-					(reference "R59")
+					(reference "R93")
 					(unit 1)
 				)
@@
 		(dnp no)
 		(fields_autoplaced yes)
-		(property "Reference" "R58"
+		(property "Reference" "R94"
 			(at 223.52 35.56 0)
 			(effects
@@
 			(project "launchpad-controller-v2"
 				(path "/8b86c7a7-6364-4b1f-ab12-b4882a7d8ae2/8c27322b-4514-4c93-94e3-74166c34f228"
-					(reference "R58")
+					(reference "R94")
 					(unit 1)
 				)
@@
 		(on_board yes)
 		(dnp no)
-		(property "Reference" "R19"
+		(property "Reference" "R90"
 			(at 35.56 60.96 90)
 			(effects
@@
 			(project "launchpad-controller-v2"
 				(path "/8b86c7a7-6364-4b1f-ab12-b4882a7d8ae2/8c27322b-4514-4c93-94e3-74166c34f228"
-					(reference "R19")
+					(reference "R90")
 					(unit 1)
 				)
@@
 		(dnp no)
 		(fields_autoplaced yes)
-		(property "Reference" "R61"
+		(property "Reference" "R91"
 			(at 222.25 90.17 0)
 			(effects
@@
 			(project "launchpad-controller-v2"
 				(path "/8b86c7a7-6364-4b1f-ab12-b4882a7d8ae2/8c27322b-4514-4c93-94e3-74166c34f228"
-					(reference "R61")
+					(reference "R91")
 					(unit 1)
 				)
@@
 		(dnp no)
 		(fields_autoplaced yes)
-		(property "Reference" "C88"
+		(property "Reference" "C1"
 			(at 240.03 86.36 0)
 			(effects
@@
 			(project "launchpad-controller-v2"
 				(path "/8b86c7a7-6364-4b1f-ab12-b4882a7d8ae2/8c27322b-4514-4c93-94e3-74166c34f228"
-					(reference "C88")
+					(reference "C1")
 					(unit 1)
 				)
@@
 		(dnp no)
 		(fields_autoplaced yes)
-		(property "Reference" "U2"
+		(property "Reference" "U32"
 			(at 101.6 24.13 0)
 			(effects
@@
 			(project "launchpad-controller-v2"
 				(path "/8b86c7a7-6364-4b1f-ab12-b4882a7d8ae2/8c27322b-4514-4c93-94e3-74166c34f228"
-					(reference "U2")
+					(reference "U32")
 					(unit 1)
 				)
