File: ina260sense.kicad_sch (KiCad schematic)
At the start: 2 parts, among them U23 INA260

Commit message: bajs
Parts:
- renumbered C122 to C6, U23 to U7
Changed lines of the file:
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@@
 		(dnp no)
 		(fields_autoplaced yes)
-		(property "Reference" "C122"
+		(property "Reference" "C6"
 			(at 78.74 33.0199 0)
 			(effects
@@
 			(project "launchpad-controller-v2"
 				(path "/8b86c7a7-6364-4b1f-ab12-b4882a7d8ae2/c6833da5-48fe-4479-a04d-d8715f8cb73f"
-					(reference "C122")
+					(reference "C6")
 					(unit 1)
 				)
 				(path "/8b86c7a7-6364-4b1f-ab12-b4882a7d8ae2/1365e2a8-987a-4458-bb6d-3c5dcf8625cf"
-					(reference "C123")
+					(reference "C56")
 					(unit 1)
 				)
 				(path "/8b86c7a7-6364-4b1f-ab12-b4882a7d8ae2/8539ee0f-bec8-42ad-ad72-6f557c8f64b7"
-					(reference "C124")
+					(reference "C27")
 					(unit 1)
 				)
@@
 		(dnp no)
 		(fields_autoplaced yes)
-		(property "Reference" "U23"
+		(property "Reference" "U7"
 			(at 88.5541 43.18 0)
 			(effects
@@
 			(project "launchpad-controller-v2"
 				(path "/8b86c7a7-6364-4b1f-ab12-b4882a7d8ae2/c6833da5-48fe-4479-a04d-d8715f8cb73f"
-					(reference "U23")
+					(reference "U7")
 					(unit 1)
 				)
 				(path "/8b86c7a7-6364-4b1f-ab12-b4882a7d8ae2/1365e2a8-987a-4458-bb6d-3c5dcf8625cf"
-					(reference "U25")
+					(reference "U22")
 					(unit 1)
 				)
 				(path "/8b86c7a7-6364-4b1f-ab12-b4882a7d8ae2/8539ee0f-bec8-42ad-ad72-6f557c8f64b7"
-					(reference "U26")
-					(unit 1)
-				)
+					(reference "U13")
+					(unit 1)
+				)
