File: power.kicad_sch (KiCad schematic)
At the start: 17 parts, among them U24 LM3940IMPX-3.3/NOPB, U27 LM2940IMPX-12/NOPB, U29 Generic Switching Reg

Commit message: bajs
Parts:
- renumbered C103 to C10, C101 to C12, C92 to C4, C91 to C5, D3 to D4, D5 to D6, D4 to D8, FB2 to FB1, R22 to R11, R24 to R14, R23 to R17, U29 to U1, U24 to U5, U27 to U8
Changed lines of the file:
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@@
 		(dnp no)
 		(fields_autoplaced yes)
-		(property "Reference" "R23"
+		(property "Reference" "R17"
 			(at 209.55 68.5799 0)
 			(effects
@@
 			(project "launchpad-controller-v2"
 				(path "/8b86c7a7-6364-4b1f-ab12-b4882a7d8ae2/4bb9601b-797d-416b-873f-14cacc30ce2a"
-					(reference "R23")
+					(reference "R17")
 					(unit 1)
 				)
@@
 		(dnp no)
 		(fields_autoplaced yes)
-		(property "Reference" "FB2"
+		(property "Reference" "FB1"
 			(at 54.5592 34.29 90)
 			(effects
@@
 			(project "launchpad-controller-v2"
 				(path "/8b86c7a7-6364-4b1f-ab12-b4882a7d8ae2/4bb9601b-797d-416b-873f-14cacc30ce2a"
-					(reference "FB2")
+					(reference "FB1")
 					(unit 1)
 				)
@@
 		(dnp no)
 		(fields_autoplaced yes)
-		(property "Reference" "U27"
+		(property "Reference" "U8"
 			(at 74.93 120.65 0)
 			(effects
@@
 			(project "launchpad-controller-v2"
 				(path "/8b86c7a7-6364-4b1f-ab12-b4882a7d8ae2/4bb9601b-797d-416b-873f-14cacc30ce2a"
-					(reference "U27")
+					(reference "U8")
 					(unit 1)
 				)
@@
 		(on_board yes)
 		(dnp no)
-		(property "Reference" "C101"
+		(property "Reference" "C12"
 			(at 52.07 147.32 0)
 			(effects
@@
 			(project "launchpad-controller-v2"
 				(path "/8b86c7a7-6364-4b1f-ab12-b4882a7d8ae2/4bb9601b-797d-416b-873f-14cacc30ce2a"
-					(reference "C101")
+					(reference "C12")
 					(unit 1)
 				)
@@
 		(dnp no)
 		(fields_autoplaced yes)
-		(property "Reference" "R22"
+		(property "Reference" "R11"
 			(at 114.3 91.44 90)
 			(effects
@@
 			(project "launchpad-controller-v2"
 				(path "/8b86c7a7-6364-4b1f-ab12-b4882a7d8ae2/4bb9601b-797d-416b-873f-14cacc30ce2a"
-					(reference "R22")
+					(reference "R11")
 					(unit 1)
 				)
@@
 		(dnp no)
 		(fields_autoplaced yes)
-		(property "Reference" "C103"
+		(property "Reference" "C10"
 			(at 106.68 147.32 0)
 			(effects
@@
 			(project "launchpad-controller-v2"
 				(path "/8b86c7a7-6364-4b1f-ab12-b4882a7d8ae2/4bb9601b-797d-416b-873f-14cacc30ce2a"
-					(reference "C103")
+					(reference "C10")
 					(unit 1)
 				)
@@
 		(dnp no)
 		(fields_autoplaced yes)
-		(property "Reference" "R24"
+		(property "Reference" "R14"
 			(at 199.39 143.5099 0)
 			(effects
@@
 			(project "launchpad-controller-v2"
 				(path "/8b86c7a7-6364-4b1f-ab12-b4882a7d8ae2/4bb9601b-797d-416b-873f-14cacc30ce2a"
-					(reference "R24")
+					(reference "R14")
 					(unit 1)
 				)
@@
 		(on_board yes)
 		(dnp no)
-		(property "Reference" "D5"
+		(property "Reference" "D6"
 			(at 189.23 136.2075 0)
 			(effects
@@
 			(project "launchpad-controller-v2"
 				(path "/8b86c7a7-6364-4b1f-ab12-b4882a7d8ae2/4bb9601b-797d-416b-873f-14cacc30ce2a"
-					(reference "D5")
+					(reference "D6")
 					(unit 1)
 				)
@@
 		(on_board yes)
 		(dnp no)
-		(property "Reference" "D4"
+		(property "Reference" "D8"
 			(at 199.39 61.2775 0)
 			(effects
@@
 			(project "launchpad-controller-v2"
 				(path "/8b86c7a7-6364-4b1f-ab12-b4882a7d8ae2/4bb9601b-797d-416b-873f-14cacc30ce2a"
-					(reference "D4")
+					(reference "D8")
 					(unit 1)
 				)
@@
 		(dnp no)
 		(fields_autoplaced yes)
-		(property "Reference" "C92"
+		(property "Reference" "C4"
 			(at 102.87 91.44 0)
 			(effects
@@
 			(project "launchpad-controller-v2"
 				(path "/8b86c7a7-6364-4b1f-ab12-b4882a7d8ae2/4bb9601b-797d-416b-873f-14cacc30ce2a"
-					(reference "C92")
+					(reference "C4")
 					(unit 1)
 				)
@@
 		(on_board yes)
 		(dnp no)
-		(property "Reference" "D3"
+		(property "Reference" "D4"
 			(at 113.03 82.8675 0)
 			(effects
@@
 			(project "launchpad-controller-v2"
 				(path "/8b86c7a7-6364-4b1f-ab12-b4882a7d8ae2/4bb9601b-797d-416b-873f-14cacc30ce2a"
-					(reference "D3")
+					(reference "D4")
 					(unit 1)
 				)
@@
 		(on_board yes)
 		(dnp no)
-		(property "Reference" "C91"
+		(property "Reference" "C5"
 			(at 45.72 86.36 0)
 			(effects
@@
 			(project "launchpad-controller-v2"
 				(path "/8b86c7a7-6364-4b1f-ab12-b4882a7d8ae2/4bb9601b-797d-416b-873f-14cacc30ce2a"
-					(reference "C91")
+					(reference "C5")
 					(unit 1)
 				)
@@
 		(on_board yes)
 		(dnp no)
-		(property "Reference" "U24"
+		(property "Reference" "U5"
 			(at 74.93 63.5 0)
 			(effects
@@
 			(project "launchpad-controller-v2"
 				(path "/8b86c7a7-6364-4b1f-ab12-b4882a7d8ae2/4bb9601b-797d-416b-873f-14cacc30ce2a"
-					(reference "U24")
+					(reference "U5")
 					(unit 1)
 				)
@@
 		(on_board yes)
 		(dnp no)
-		(property "Reference" "U29"
+		(property "Reference" "U1"
 			(at 97.79 47.6251 0)
 			(effects
@@
 			(project "launchpad-controller-v2"
 				(path "/8b86c7a7-6364-4b1f-ab12-b4882a7d8ae2/4bb9601b-797d-416b-873f-14cacc30ce2a"
-					(reference "U29")
-					(unit 1)
-				)
+					(reference "U1")
+					(unit 1)
+				)
