File: thermocouple.kicad_sch (KiCad schematic)
At the start: 12 parts, among them U1 AD8495

Commit message: bajs
Parts:
- renumbered C4 to C42, C2 to C46, C8 to C50, C6 to C89, C7 to C90, C3 to C93, R99 to R40, R91 to R43, R2 to R56, R1 to R96, TC1 to TC6, U1 to U19
Other:
- note added: "Might need decoupling cap on VS-"
