File: voltage_input_filtering.kicad_sch (KiCad schematic)
At the start: 4 parts, among them J22 Conn_01x04

Commit message: bajs
Parts:
- renumbered C93 to C23, D1 to D21, J22 to J21, R69 to R37
Changed lines of the file:
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@@
 		(dnp no)
 		(fields_autoplaced yes)
-		(property "Reference" "C93"
+		(property "Reference" "C23"
 			(at 106.68 63.5 0)
 			(effects
@@
 			(project "launchpad-controller-v2"
 				(path "/8b86c7a7-6364-4b1f-ab12-b4882a7d8ae2/dbac82f3-7447-480a-94cd-632941520571/400639c7-67af-4359-b7ea-5963132c438d"
-					(reference "C93")
+					(reference "C23")
 					(unit 1)
 				)
 				(path "/8b86c7a7-6364-4b1f-ab12-b4882a7d8ae2/dbac82f3-7447-480a-94cd-632941520571/b8c8e7ad-e483-4f1e-a921-619fd227ce2a"
-					(reference "C94")
+					(reference "C14")
 					(unit 1)
 				)
 				(path "/8b86c7a7-6364-4b1f-ab12-b4882a7d8ae2/dbac82f3-7447-480a-94cd-632941520571/bef595c2-0dbc-4b04-a8d4-4a9a80018c48"
-					(reference "C95")
+					(reference "C13")
 					(unit 1)
 				)
 				(path "/8b86c7a7-6364-4b1f-ab12-b4882a7d8ae2/dbac82f3-7447-480a-94cd-632941520571/7007d3c3-03b9-4564-8f31-2f57c9a50e16"
-					(reference "C96")
+					(reference "C26")
 					(unit 1)
 				)
 				(path "/8b86c7a7-6364-4b1f-ab12-b4882a7d8ae2/5b962238-ad91-40ff-b76d-985e2dbc0aeb/400639c7-67af-4359-b7ea-5963132c438d"
-					(reference "C97")
+					(reference "C7")
 					(unit 1)
 				)
 				(path "/8b86c7a7-6364-4b1f-ab12-b4882a7d8ae2/5b962238-ad91-40ff-b76d-985e2dbc0aeb/bef595c2-0dbc-4b04-a8d4-4a9a80018c48"
-					(reference "C98")
+					(reference "C9")
 					(unit 1)
 				)
 				(path "/8b86c7a7-6364-4b1f-ab12-b4882a7d8ae2/5b962238-ad91-40ff-b76d-985e2dbc0aeb/7007d3c3-03b9-4564-8f31-2f57c9a50e16"
-					(reference "C99")
+					(reference "C11")
 					(unit 1)
 				)
 				(path "/8b86c7a7-6364-4b1f-ab12-b4882a7d8ae2/5b962238-ad91-40ff-b76d-985e2dbc0aeb/b8c8e7ad-e483-4f1e-a921-619fd227ce2a"
-					(reference "C100")
+					(reference "C8")
 					(unit 1)
 				)
@@
 		(dnp no)
 		(fields_autoplaced yes)
-		(property "Reference" "D1"
+		(property "Reference" "D21"
 			(at 72.39 63.5 90)
 			(effects
@@
 			(project "launchpad-controller-v2"
 				(path "/8b86c7a7-6364-4b1f-ab12-b4882a7d8ae2/dbac82f3-7447-480a-94cd-632941520571/400639c7-67af-4359-b7ea-5963132c438d"
-					(reference "D1")
+					(reference "D21")
 					(unit 1)
 				)
 				(path "/8b86c7a7-6364-4b1f-ab12-b4882a7d8ae2/dbac82f3-7447-480a-94cd-632941520571/b8c8e7ad-e483-4f1e-a921-619fd227ce2a"
-					(reference "D2")
+					(reference "D18")
 					(unit 1)
 				)
 				(path "/8b86c7a7-6364-4b1f-ab12-b4882a7d8ae2/dbac82f3-7447-480a-94cd-632941520571/bef595c2-0dbc-4b04-a8d4-4a9a80018c48"
-					(reference "D23")
+					(reference "D17")
 					(unit 1)
 				)
 				(path "/8b86c7a7-6364-4b1f-ab12-b4882a7d8ae2/dbac82f3-7447-480a-94cd-632941520571/7007d3c3-03b9-4564-8f31-2f57c9a50e16"
-					(reference "D24")
+					(reference "D20")
 					(unit 1)
 				)
 				(path "/8b86c7a7-6364-4b1f-ab12-b4882a7d8ae2/5b962238-ad91-40ff-b76d-985e2dbc0aeb/400639c7-67af-4359-b7ea-5963132c438d"
-					(reference "D25")
+					(reference "D13")
 					(unit 1)
 				)
 				(path "/8b86c7a7-6364-4b1f-ab12-b4882a7d8ae2/5b962238-ad91-40ff-b76d-985e2dbc0aeb/bef595c2-0dbc-4b04-a8d4-4a9a80018c48"
-					(reference "D26")
+					(reference "D16")
 					(unit 1)
 				)
 				(path "/8b86c7a7-6364-4b1f-ab12-b4882a7d8ae2/5b962238-ad91-40ff-b76d-985e2dbc0aeb/7007d3c3-03b9-4564-8f31-2f57c9a50e16"
-					(reference "D27")
+					(reference "D15")
 					(unit 1)
 				)
 				(path "/8b86c7a7-6364-4b1f-ab12-b4882a7d8ae2/5b962238-ad91-40ff-b76d-985e2dbc0aeb/b8c8e7ad-e483-4f1e-a921-619fd227ce2a"
-					(reference "D28")
+					(reference "D14")
 					(unit 1)
 				)
@@
 		(dnp no)
 		(fields_autoplaced yes)
-		(property "Reference" "J22"
+		(property "Reference" "J21"
 			(at 48.26 49.53 0)
 			(effects
@@
 			(project "launchpad-controller-v2"
 				(path "/8b86c7a7-6364-4b1f-ab12-b4882a7d8ae2/dbac82f3-7447-480a-94cd-632941520571/400639c7-67af-4359-b7ea-5963132c438d"
-					(reference "J22")
+					(reference "J21")
 					(unit 1)
 				)
 				(path "/8b86c7a7-6364-4b1f-ab12-b4882a7d8ae2/dbac82f3-7447-480a-94cd-632941520571/b8c8e7ad-e483-4f1e-a921-619fd227ce2a"
-					(reference "J24")
+					(reference "J13")
 					(unit 1)
 				)
 				(path "/8b86c7a7-6364-4b1f-ab12-b4882a7d8ae2/dbac82f3-7447-480a-94cd-632941520571/bef595c2-0dbc-4b04-a8d4-4a9a80018c48"
-					(reference "J25")
+					(reference "J14")
 					(unit 1)
 				)
 				(path "/8b86c7a7-6364-4b1f-ab12-b4882a7d8ae2/dbac82f3-7447-480a-94cd-632941520571/7007d3c3-03b9-4564-8f31-2f57c9a50e16"
-					(reference "J26")
+					(reference "J23")
 					(unit 1)
 				)
 				(path "/8b86c7a7-6364-4b1f-ab12-b4882a7d8ae2/5b962238-ad91-40ff-b76d-985e2dbc0aeb/400639c7-67af-4359-b7ea-5963132c438d"
-					(reference "J27")
+					(reference "J10")
 					(unit 1)
 				)
 				(path "/8b86c7a7-6364-4b1f-ab12-b4882a7d8ae2/5b962238-ad91-40ff-b76d-985e2dbc0aeb/bef595c2-0dbc-4b04-a8d4-4a9a80018c48"
-					(reference "J28")
+					(reference "J12")
 					(unit 1)
 				)
 				(path "/8b86c7a7-6364-4b1f-ab12-b4882a7d8ae2/5b962238-ad91-40ff-b76d-985e2dbc0aeb/7007d3c3-03b9-4564-8f31-2f57c9a50e16"
-					(reference "J29")
+					(reference "J11")
 					(unit 1)
 				)
 				(path "/8b86c7a7-6364-4b1f-ab12-b4882a7d8ae2/5b962238-ad91-40ff-b76d-985e2dbc0aeb/b8c8e7ad-e483-4f1e-a921-619fd227ce2a"
-					(reference "J30")
+					(reference "J9")
 					(unit 1)
 				)
@@
 		(dnp no)
 		(fields_autoplaced yes)
-		(property "Reference" "R69"
+		(property "Reference" "R37"
 			(at 87.63 54.61 90)
 			(effects
@@
 			(project "launchpad-controller-v2"
 				(path "/8b86c7a7-6364-4b1f-ab12-b4882a7d8ae2/dbac82f3-7447-480a-94cd-632941520571/400639c7-67af-4359-b7ea-5963132c438d"
-					(reference "R69")
+					(reference "R37")
 					(unit 1)
 				)
 				(path "/8b86c7a7-6364-4b1f-ab12-b4882a7d8ae2/dbac82f3-7447-480a-94cd-632941520571/b8c8e7ad-e483-4f1e-a921-619fd227ce2a"
-					(reference "R70")
+					(reference "R30")
 					(unit 1)
 				)
 				(path "/8b86c7a7-6364-4b1f-ab12-b4882a7d8ae2/dbac82f3-7447-480a-94cd-632941520571/bef595c2-0dbc-4b04-a8d4-4a9a80018c48"
-					(reference "R71")
+					(reference "R29")
 					(unit 1)
 				)
 				(path "/8b86c7a7-6364-4b1f-ab12-b4882a7d8ae2/dbac82f3-7447-480a-94cd-632941520571/7007d3c3-03b9-4564-8f31-2f57c9a50e16"
-					(reference "R72")
+					(reference "R36")
 					(unit 1)
 				)
 				(path "/8b86c7a7-6364-4b1f-ab12-b4882a7d8ae2/5b962238-ad91-40ff-b76d-985e2dbc0aeb/400639c7-67af-4359-b7ea-5963132c438d"
-					(reference "R73")
+					(reference "R25")
 					(unit 1)
 				)
 				(path "/8b86c7a7-6364-4b1f-ab12-b4882a7d8ae2/5b962238-ad91-40ff-b76d-985e2dbc0aeb/bef595c2-0dbc-4b04-a8d4-4a9a80018c48"
-					(reference "R74")
+					(reference "R28")
 					(unit 1)
 				)
 				(path "/8b86c7a7-6364-4b1f-ab12-b4882a7d8ae2/5b962238-ad91-40ff-b76d-985e2dbc0aeb/7007d3c3-03b9-4564-8f31-2f57c9a50e16"
-					(reference "R75")
+					(reference "R27")
 					(unit 1)
 				)
 				(path "/8b86c7a7-6364-4b1f-ab12-b4882a7d8ae2/5b962238-ad91-40ff-b76d-985e2dbc0aeb/b8c8e7ad-e483-4f1e-a921-619fd227ce2a"
-					(reference "R76")
-					(unit 1)
-				)
+					(reference "R26")
+					(unit 1)
+				)
